File: hfamp.sch (KiCad schematic (older format))
At the start: 20 parts, among them K1 CONN_3, P1 CONN_2, Q1 DARL_N, U1 7805

Commit message: Finished schematic.
Parts:
- added C10, C12, C13: .1u, symbol C
- added C11, C8, C9: .01u, symbol C
- added C14, C15: 110p, symbol C
- added D5, D6: DIODE, symbol DIODE
- added L2, L3: RFC, symbol INDUCTOR
- added L4: .53u, symbol INDUCTOR
- added P2, P3: CONN_2, symbol CONN_2
- added Q2: MOSFET_N, symbol MOSFET_N
- added R3, R5: 330, symbol R
- added R4: 18, symbol R
- added R6: 51, symbol R
- added R7, R8: 1k, symbol R
- added R9: 10, symbol R
- added T1: 1:2.6, symbol TRANSFO
Connections:
- wire segments 32 -> 51
Other:
- note added: "10W Amplifier"

Commit message: Forgot to label MOSFET as IRF510.
Parts:
- Q2: value MOSFET_N -> IRF510
Changed lines of the file:
@@
-EESchema Schematic File Version 2  date Sat 07 Dec 2013 10:31:43 AM CST
+EESchema Schematic File Version 2  date Sat 07 Dec 2013 11:36:14 AM CST
 LIBS:power
 LIBS:device
@@
 P 8500 2450
 F 0 "Q2" H 8510 2620 60  0000 R CNN
-F 1 "MOSFET_N" H 8510 2300 60  0000 R CNN
+F 1 "IRF510" H 8510 2300 60  0000 R CNN
 	1    8500 2450
 	1    0    0    -1

Commit message: Added footprints for each component.
Ready to start laying out the board.
Parts:
- D2, D3: value DIODE -> BAT62-03W
- D4, D5, D6: value DIODE -> 1N4148W
- Q1: value DARL_N -> MMBT6427
Changed lines of the file:
@@
-EESchema Schematic File Version 2  date Sat 07 Dec 2013 11:36:14 AM CST
+EESchema Schematic File Version 2  date Sat 07 Dec 2013 04:25:28 PM CST
 LIBS:power
 LIBS:device
@@
 10W Amplifier
 $Comp
-L GND #PWR26
+L GND #PWR01
 U 1 1 52A34B89
 P 10600 2950
-F 0 "#PWR26" H 10600 2950 30  0001 C CNN
+F 0 "#PWR01" H 10600 2950 30  0001 C CNN
 F 1 "GND" H 10600 2880 30  0001 C CNN
 	1    10600 2950
@@
 $EndComp
 $Comp
-L GND #PWR25
+L GND #PWR02
 U 1 1 52A34B85
 P 10000 2950
-F 0 "#PWR25" H 10000 2950 30  0001 C CNN
+F 0 "#PWR02" H 10000 2950 30  0001 C CNN
 F 1 "GND" H 10000 2880 30  0001 C CNN
 	1    10000 2950
@@
 $EndComp
 $Comp
-L GND #PWR24
+L GND #PWR03
 U 1 1 52A34B82
 P 9800 2950
-F 0 "#PWR24" H 9800 2950 30  0001 C CNN
+F 0 "#PWR03" H 9800 2950 30  0001 C CNN
 F 1 "GND" H 9800 2880 30  0001 C CNN
 	1    9800 2950
@@
 $EndComp
 $Comp
-L GND #PWR23
+L GND #PWR04
 U 1 1 52A34B7F
 P 9000 2950
-F 0 "#PWR23" H 9000 2950 30  0001 C CNN
+F 0 "#PWR04" H 9000 2950 30  0001 C CNN
 F 1 "GND" H 9000 2880 30  0001 C CNN
 	1    9000 2950
@@
 $EndComp
 $Comp
-L GND #PWR22
+L GND #PWR05
 U 1 1 52A34B7A
 P 8600 2950
-F 0 "#PWR22" H 8600 2950 30  0001 C CNN
+F 0 "#PWR05" H 8600 2950 30  0001 C CNN
 F 1 "GND" H 8600 2880 30  0001 C CNN
 	1    8600 2950
@@
 VDD
 $Comp
-L GND #PWR21
+L GND #PWR06
 U 1 1 52A349AA
 P 8200 1350
-F 0 "#PWR21" H 8200 1350 30  0001 C CNN
+F 0 "#PWR06" H 8200 1350 30  0001 C CNN
 F 1 "GND" H 8200 1280 30  0001 C CNN
 	1    8200 1350
@@
 $EndComp
 $Comp
-L GND #PWR20
+L GND #PWR07
 U 1 1 52A349A6
 P 8200 1100
-F 0 "#PWR20" H 8200 1100 30  0001 C CNN
+F 0 "#PWR07" H 8200 1100 30  0001 C CNN
 F 1 "GND" H 8200 1030 30  0001 C CNN
 	1    8200 1100
@@
 $EndComp
 $Comp
-L GND #PWR18
+L GND #PWR08
 U 1 1 52A34999
 P 6950 1100
-F 0 "#PWR18" H 6950 1100 30  0001 C CNN
+F 0 "#PWR08" H 6950 1100 30  0001 C CNN
 F 1 "GND" H 6950 1030 30  0001 C CNN
 	1    6950 1100
@@
 $EndComp
 $Comp
-L GND #PWR19
+L GND #PWR09
 U 1 1 52A34994
 P 6950 1350
-F 0 "#PWR19" H 6950 1350 30  0001 C CNN
+F 0 "#PWR09" H 6950 1350 30  0001 C CNN
 F 1 "GND" H 6950 1280 30  0001 C CNN
 	1    6950 1350
@@
 $EndComp
 $Comp
-L GND #PWR17
+L GND #PWR010
 U 1 1 52A34976
 P 6750 2950
-F 0 "#PWR17" H 6750 2950 30  0001 C CNN
+F 0 "#PWR010" H 6750 2950 30  0001 C CNN
 F 1 "GND" H 6750 2880 30  0001 C CNN
 	1    6750 2950
@@
 $EndComp
 $Comp
-L GND #PWR16
+L GND #PWR011
 U 1 1 52A34972
 P 6500 2950
-F 0 "#PWR16" H 6500 2950 30  0001 C CNN
+F 0 "#PWR011" H 6500 2950 30  0001 C CNN
 F 1 "GND" H 6500 2880 30  0001 C CNN
 	1    6500 2950
@@
 $EndComp
 $Comp
-L GND #PWR15
+L GND #PWR012
 U 1 1 52A34965
 P 6000 2950
-F 0 "#PWR15" H 6000 2950 30  0001 C CNN
+F 0 "#PWR012" H 6000 2950 30  0001 C CNN
 F 1 "GND" H 6000 2880 30  0001 C CNN
 	1    6000 2950
@@
 P 8400 1100
 F 0 "D6" H 8400 1200 40  0000 C CNN
-F 1 "DIODE" H 8400 1000 40  0000 C CNN
+F 1 "1N4148W" H 8400 1000 40  0000 C CNN
 	1    8400 1100
 	1    0    0    -1
@@
 P 7150 1100
 F 0 "D5" H 7150 1200 40  0000 C CNN
-F 1 "DIODE" H 7150 1000 40  0000 C CNN
+F 1 "1N4148W" H 7150 1000 40  0000 C CNN
 	1    7150 1100
 	1    0    0    -1
@@
 vbias
 $Comp
-L GND #PWR9
+L GND #PWR013
 U 1 1 52A333B8
 P 2300 4450
-F 0 "#PWR9" H 2300 4450 30  0001 C CNN
+F 0 "#PWR013" H 2300 4450 30  0001 C CNN
 F 1 "GND" H 2300 4380 30  0001 C CNN
 	1    2300 4450
@@
 $EndComp
 $Comp
-L GND #PWR7
+L GND #PWR014
 U 1 1 52A333B4
 P 1900 4450
-F 0 "#PWR7" H 1900 4450 30  0001 C CNN
+F 0 "#PWR014" H 1900 4450 30  0001 C CNN
 F 1 "GND" H 1900 4380 30  0001 C CNN
 	1    1900 4450
@@
 $EndComp
 $Comp
-L GND #PWR3
+L GND #PWR015
 U 1 1 52A333B0
 P 1500 4450
-F 0 "#PWR3" H 1500 4450 30  0001 C CNN
+F 0 "#PWR015" H 1500 4450 30  0001 C CNN
 F 1 "GND" H 1500 4380 30  0001 C CNN
 	1    1500 4450
@@
 $EndComp
 $Comp
-L GND #PWR1
+L GND #PWR016
 U 1 1 52A333A7
 P 1100 4450
-F 0 "#PWR1" H 1100 4450 30  0001 C CNN
+F 0 "#PWR016" H 1100 4450 30  0001 C CNN
 F 1 "GND" H 1100 4380 30  0001 C CNN
 	1    1100 4450
@@
 $EndComp
 $Comp
-L +5V #PWR6
+L +5V #PWR017
 U 1 1 52A3339C
 P 1900 3800
-F 0 "#PWR6" H 1900 3890 20  0001 C CNN
+F 0 "#PWR017" H 1900 3890 20  0001 C CNN
 F 1 "+5V" H 1900 3890 30  0000 C CNN
 	1    1900 3800
@@
 P 3200 2850
 F 0 "D4" H 3200 2950 40  0000 C CNN
-F 1 "DIODE" H 3200 2750 40  0000 C CNN
+F 1 "1N4148W" H 3200 2750 40  0000 C CNN
 	1    3200 2850
 	0    1    1    0
 $EndComp
 $Comp
-L +5V #PWR13
+L +5V #PWR018
 U 1 1 52A330A3
 P 3300 3250
-F 0 "#PWR13" H 3300 3340 20  0001 C CNN
+F 0 "#PWR018" H 3300 3340 20  0001 C CNN
 F 1 "+5V" H 3300 3340 30  0000 C CNN
 	1    3300 3250
@@
 $EndComp
 $Comp
-L GND #PWR12
+L GND #PWR019
 U 1 1 52A32C37
 P 3000 3250
-F 0 "#PWR12" H 3000 3250 30  0001 C CNN
+F 0 "#PWR019" H 3000 3250 30  0001 C CNN
 F 1 "GND" H 3000 3180 30  0001 C CNN
 	1    3000 3250
@@
 $EndComp
 $Comp
-L GND #PWR8
+L GND #PWR020
 U 1 1 52A32C1F
 P 2200 3250
-F 0 "#PWR8" H 2200 3250 30  0001 C CNN
+F 0 "#PWR020" H 2200 3250 30  0001 C CNN
 F 1 "GND" H 2200 3180 30  0001 C CNN
 	1    2200 3250
@@
 $EndComp
 $Comp
-L GND #PWR5
+L GND #PWR021
 U 1 1 52A32C1A
 P 1800 3250
-F 0 "#PWR5" H 1800 3250 30  0001 C CNN
+F 0 "#PWR021" H 1800 3250 30  0001 C CNN
 F 1 "GND" H 1800 3180 30  0001 C CNN
 	1    1800 3250
@@
 P 2750 2900
 F 0 "Q1" H 2750 3150 50  0000 C CNN
-F 1 "DARL_N" H 2550 2800 50  0000 C CNN
+F 1 "MMBT6427" H 2550 2800 50  0000 C CNN
 	1    2750 2900
 	1    0    0    -1
@@
 P 2000 2850
 F 0 "D3" H 2000 2950 40  0000 C CNN
-F 1 "DIODE" H 2000 2750 40  0000 C CNN
+F 1 "BAT62-03W" H 2000 2750 40  0000 C CNN
 	1    2000 2850
 	1    0    0    -1
@@
 P 1800 3050
 F 0 "D2" H 1800 3150 40  0000 C CNN
-F 1 "DIODE" H 1800 2950 40  0000 C CNN
+F 1 "BAT62-03W" H 1800 2950 40  0000 C CNN
 	1    1800 3050
 	0    -1   -1   0
@@
 VDD
 $Comp
-L GND #PWR14
+L GND #PWR022
 U 1 1 52A10FBB
 P 3400 2100
-F 0 "#PWR14" H 3400 2100 30  0001 C CNN
+F 0 "#PWR022" H 3400 2100 30  0001 C CNN
 F 1 "GND" H 3400 2030 30  0001 C CNN
 	1    3400 2100
@@
 $EndComp
 $Comp
-L GND #PWR11
+L GND #PWR023
 U 1 1 52A10FB8
 P 2850 2100
-F 0 "#PWR11" H 2850 2100 30  0001 C CNN
+F 0 "#PWR023" H 2850 2100 30  0001 C CNN
 F 1 "GND" H 2850 2030 30  0001 C CNN
 	1    2850 2100
@@
 $EndComp
 $Comp
-L GND #PWR10
+L GND #PWR024
 U 1 1 52A10FB3
 P 2500 2100
-F 0 "#PWR10" H 2500 2100 30  0001 C CNN
+F 0 "#PWR024" H 2500 2100 30  0001 C CNN
 F 1 "GND" H 2500 2030 30  0001 C CNN
 	1    2500 2100
@@
 $EndComp
 $Comp
-L GND #PWR4
+L GND #PWR025
 U 1 1 52A10FAF
 P 1800 2100
-F 0 "#PWR4" H 1800 2100 30  0001 C CNN
+F 0 "#PWR025" H 1800 2100 30  0001 C CNN
 F 1 "GND" H 1800 2030 30  0001 C CNN
 	1    1800 2100
@@
 $EndComp
 $Comp
-L GND #PWR2
+L GND #PWR026
 U 1 1 52A10FA4
 P 1250 2100
-F 0 "#PWR2" H 1250 2100 30  0001 C CNN
+F 0 "#PWR026" H 1250 2100 30  0001 C CNN
 F 1 "GND" H 1250 2030 30  0001 C CNN
 	1    1250 2100

Commit message: Finished board layout.
Connections:
- wire segments 51 -> 53
Other:
- moved on the sheet: D4
Changed lines of the file:
@@
-EESchema Schematic File Version 2  date Sat 07 Dec 2013 04:25:28 PM CST
+EESchema Schematic File Version 2  date Sat 07 Dec 2013 06:45:23 PM CST
 LIBS:power
 LIBS:device
@@
 Sheet 1 1
 Title "HF Amp: 0.5W to 10W"
-Date "7 dec 2013"
+Date "8 dec 2013"
 Rev "1.2"
 Comp ""
@@
 Comment4 ""
 $EndDescr
+Connection ~ 7600 2450
+Connection ~ 7350 2450
+Connection ~ 3150 3150
+Wire Wire Line
+	3050 3150 3300 3150
+Wire Wire Line
+	3050 3150 3050 2650
+Wire Wire Line
+	3050 2650 2900 2650
+Wire Wire Line
+	3150 2750 3300 2750
+Wire Wire Line
+	4450 3600 4550 3600
+Wire Wire Line
+	4450 3800 4450 4050
+Wire Notes Line
+	11150 3050 5200 3050
+Wire Notes Line
+	11150 3050 11150 550
+Wire Notes Line
+	11150 550  5200 550
+Wire Notes Line
+	5200 550  5200 3050
+Wire Wire Line
+	10600 2650 10600 2950
+Wire Wire Line
+	9800 2250 10000 2250
+Wire Wire Line
+	9000 2650 9000 2950
+Wire Wire Line
+	5600 2450 5500 2450
+Connection ~ 7350 1100
+Wire Wire Line
+	7350 950  7350 1350
+Wire Wire Line
+	7600 1950 7850 1950
+Wire Wire Line
+	6500 2450 6750 2450
+Wire Wire Line
+	2450 4200 2600 4200
+Wire Wire Line
+	1100 3950 900  3950
+Wire Wire Line
+	1500 4250 1500 4450
+Wire Wire Line
+	2300 3950 1900 3950
+Wire Wire Line
+	4200 2650 4600 2650
+Wire Wire Line
+	4200 3150 4300 3150
+Wire Wire Line
+	4300 3150 4300 2850
+Wire Wire Line
+	4300 2850 4200 2850
+Wire Wire Line
+	4200 2750 4350 2750
+Wire Wire Line
+	3000 3050 3000 3250
+Wire Wire Line
+	1250 2100 1250 1200
+Wire Wire Line
+	1250 1200 1150 1200
+Wire Wire Line
+	1300 1300 1300 1100
+Wire Wire Line
+	1300 1300 1150 1300
+Wire Wire Line
+	4550 1100 4250 1100
+Wire Wire Line
+	2850 1500 2850 2100
+Connection ~ 2850 1100
+Wire Wire Line
+	2500 2050 2500 2100
+Wire Wire Line
+	1800 1500 1800 2100
+Connection ~ 1800 1100
+Wire Wire Line
+	2500 1500 2500 1550
+Connection ~ 2500 1100
+Wire Wire Line
+	2300 1100 3650 1100
+Connection ~ 3400 1100
+Wire Wire Line
+	3400 1500 3400 2100
+Wire Notes Line
+	600  2250 600  550
+Wire Notes Line
+	600  2250 5050 2250
+Wire Notes Line
+	5050 2250 5050 550
+Wire Notes Line
+	5050 550  600  550
+Wire Wire Line
+	1300 1100 2100 1100
+Wire Wire Line
+	2200 2850 2500 2850
+Wire Wire Line
+	4200 3050 4350 3050
+Wire Wire Line
+	4200 2950 4600 2950
+Wire Notes Line
+	4900 2400 600  2400
+Wire Notes Line
+	4900 2400 4900 3400
+Wire Notes Line
+	4900 3400 600  3400
+Wire Notes Line
+	600  3400 600  2400
+Wire Wire Line
+	1900 4350 1900 4450
+Wire Wire Line
+	1100 4350 1100 4450
+Wire Wire Line
+	1900 3950 1900 3800
+Wire Notes Line
+	2950 3550 600  3550
+Wire Notes Line
+	2950 3550 2950 4550
+Wire Notes Line
+	2950 4550 600  4550
+Wire Notes Line
+	600  4550 600  3550
+Wire Wire Line
+	7150 2450 7800 2450
+Wire Wire Line
+	8250 1950 8600 1950
+Wire Wire Line
+	8600 1950 8600 2250
+Wire Wire Line
+	8600 950  8600 1350
+Connection ~ 8600 1100
+Wire Wire Line
+	8600 2650 8600 2950
+Wire Wire Line
+	9800 2650 9800 2950
+Wire Wire Line
+	10000 2650 10000 2950
+Wire Wire Line
+	10600 2250 10900 2250
+Wire Wire Line
+	3600 3800 3600 4050
+Wire Wire Line
+	3600 3600 3700 3600
+Wire Wire Line
+	3300 2750 3300 2550
+Wire Wire Line
+	3300 3150 3300 3050
 Text GLabel 4550 3600 2    60   Input ~ 0
 vout
 Text GLabel 3700 3600 2    60   Input ~ 0
 vin
-Wire Wire Line
-	4450 3600 4550 3600
-Wire Wire Line
-	4450 3800 4450 4050
-Wire Notes Line
-	11150 3050 5200 3050
-Wire Notes Line
-	11150 3050 11150 550
-Wire Notes Line
-	11150 550  5200 550
-Wire Notes Line
-	5200 550  5200 3050
-Wire Wire Line
-	10600 2650 10600 2950
-Wire Wire Line
-	9800 2250 10000 2250
-Wire Wire Line
-	9000 2650 9000 2950
-Wire Wire Line
-	5600 2450 5500 2450
-Connection ~ 7350 1100
-Wire Wire Line
-	7350 950  7350 1350
-Wire Wire Line
-	7600 1950 7850 1950
-Wire Wire Line
-	6500 2450 6750 2450
-Wire Wire Line
-	2450 4200 2600 4200
-Wire Wire Line
-	1100 3950 900  3950
-Wire Wire Line
-	1500 4250 1500 4450
-Wire Wire Line
-	2300 3950 1900 3950
-Wire Wire Line
-	4200 2650 4600 2650
-Wire Wire Line
-	4200 3150 4300 3150
-Wire Wire Line
-	4300 3150 4300 2850
-Wire Wire Line
-	4300 2850 4200 2850
-Wire Wire Line
-	4200 2750 4350 2750
-Wire Wire Line
-	3300 3250 3300 3050
-Wire Wire Line
-	3000 3050 3000 3250
-Wire Wire Line
-	1250 2100 1250 1200
-Wire Wire Line
-	1250 1200 1150 1200
-Wire Wire Line
-	1300 1300 1300 1100
-Wire Wire Line
-	1300 1300 1150 1300
-Wire Wire Line
-	4550 1100 4250 1100
-Wire Wire Line
-	2850 1500 2850 2100
-Connection ~ 2850 1100
-Wire Wire Line
-	2500 2050 2500 2100
-Wire Wire Line
-	1800 1500 1800 2100
-Connection ~ 1800 1100
-Wire Wire Line
-	2500 1500 2500 1550
-Connection ~ 2500 1100
-Wire Wire Line
-	2300 1100 3650 1100
-Connection ~ 3400 1100
-Wire Wire Line
-	3400 1500 3400 2100
-Wire Notes Line
-	600  2250 600  550
-Wire Notes Line
-	600  2250 5050 2250
-Wire Notes Line
-	5050 2250 5050 550
-Wire Notes Line
-	5050 550  600  550
-Wire Wire Line
-	1300 1100 2100 1100
-Wire Wire Line
-	2200 2850 2500 2850
-Wire Wire Line
-	2900 2650 3300 2650
-Wire Wire Line
-	3300 2650 3300 2750
-Wire Wire Line
-	3300 3050 3200 3050
-Wire Wire Line
-	4200 3050 4350 3050
-Wire Wire Line
-	4200 2950 4600 2950
-Wire Notes Line
-	4900 2400 600  2400
-Wire Notes Line
-	4900 2400 4900 3400
-Wire Notes Line
-	4900 3400 600  3400
-Wire Notes Line
-	600  3400 600  2400
-Wire Wire Line
-	1900 4350 1900 4450
-Wire Wire Line
-	1100 4350 1100 4450
-Wire Wire Line
-	1900 3950 1900 3800
-Wire Notes Line
-	2950 3550 600  3550
-Wire Notes Line
-	2950 3550 2950 4550
-Wire Notes Line
-	2950 4550 600  4550
-Wire Notes Line
-	600  4550 600  3550
-Wire Wire Line
-	7150 2450 7800 2450
-Wire Wire Line
-	8250 1950 8600 1950
-Wire Wire Line
-	8600 1950 8600 2250
-Wire Wire Line
-	8600 950  8600 1350
-Connection ~ 8600 1100
-Wire Wire Line
-	8600 2650 8600 2950
-Wire Wire Line
-	9800 2650 9800 2950
-Wire Wire Line
-	10000 2650 10000 2950
-Wire Wire Line
-	10600 2250 10900 2250
-Wire Wire Line
-	3600 3800 3600 4050
-Wire Wire Line
-	3600 3600 3700 3600
 $Comp
 L CONN_2 P3
@@
 L DIODE D4
 U 1 1 52A330BE
-P 3200 2850
-F 0 "D4" H 3200 2950 40  0000 C CNN
-F 1 "1N4148W" H 3200 2750 40  0000 C CNN
-	1    3200 2850
-	0    1    1    0
+P 3150 2950
+F 0 "D4" H 3150 3050 40  0000 C CNN
+F 1 "1N4148W" H 3150 2850 40  0000 C CNN
+	1    3150 2950
+	0    -1   -1   0
 $EndComp
 $Comp
 L +5V #PWR018
 U 1 1 52A330A3
-P 3300 3250
-F 0 "#PWR018" H 3300 3340 20  0001 C CNN
-F 1 "+5V" H 3300 3340 30  0000 C CNN
-	1    3300 3250
-	-1   0    0    1
-$EndComp
-$Comp
+P 3300 2550
+F 0 "#PWR018" H 3300 2640 20  0001 C CNN
+F 1 "+5V" H 3300 2640 30  0000 C CNN
+	1    3300 2550
+	1    0    0    -1
+$EndComp
+$Comp
